Commit message: avoid using substitution

File: vnoid_challenge/model/field2023_athletics.urdf (robot description, URDF)
Before this commit: robot HVAC2023_athletics_field, 10 links, 9 joints
Links:
- link Base: geometry collision mesh filename=../../../../choreonoid/share/choreonoid-2.2/model/field2023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; collision mesh filename=../../../../choreonoid/share/choreonoid-2.2/model/field2023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
- link Link1: geometry collision box size=0.04 0.04 1.03; visual mesh filename=../../../../choreonoid/share/choreonoid-2.2/model/field2023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
- link Link2: geometry collision box size=0.04 0.04 1.03; visual mesh filename=../../../../choreonoid/share/choreonoid-2.2/model/field2023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
- link Link3: geometry collision box size=0.04 0.04 1.03; visual mesh filename=../../../../choreonoid/share/choreonoid-2.2/model/field2023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
- link Link4: geometry collision box size=0.04 0.04 1.03; visual mesh filename=../../../../choreonoid/share/choreonoid-2.2/model/field2023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
- link MovablePlate: geometry collision box size=3.0 0.7 0.1; visual mesh filename=../../../../choreonoid/share/choreonoid-2.2/model/field2023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
- link Prop1: geometry visual mesh filename=../../../../choreonoid/share/choreonoid-2.2/model/field2023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
- link Prop2: geometry visual mesh filename=../../../../choreonoid/share/choreonoid-2.2/model/field2023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
- link Prop3: geometry visual mesh filename=../../../../choreonoid/share/choreonoid-2.2/model/field2023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
- link Prop4: geometry visual mesh filename=../../../../choreonoid/share/choreonoid-2.2/model/field2023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
Joints:
- joint Link1_joint: limit lower=${radians(-90)} upper=${radians(90)} effort=100 velocity=1.0 -> lower=-1.5707 upper=1.5707 effort=100 velocity=1.0
- joint Link2_joint: limit lower=${radians(-90)} upper=${radians(90)} effort=100 velocity=1.0 -> lower=-1.5707 upper=1.5707 effort=100 velocity=1.0
- joint Link3_joint: limit lower=${radians(-90)} upper=${radians(90)} effort=100 velocity=1.0 -> lower=-1.5707 upper=1.5707 effort=100 velocity=1.0
- joint Link4_joint: limit lower=${radians(-90)} upper=${radians(90)} effort=100 velocity=1.0 -> lower=-1.5707 upper=1.5707 effort=100 velocity=1.0
